Commit message: Use box collision primitive for epick_body
Replaces the cylinder (r=0.044, l=0.1023) with a box (X=0.1025,
Y=0.075, Z=0.115) for the EPick body's collision geometry. The
visual mesh and the body_length kinematic offset are unchanged;
only the collision shape differs. The box is centered at the
body link origin like the previous cylinder.

File: epick_description/urdf/epick_body.xacro (robot description, xacro)
@@ -24,5 +24,5 @@
     <xacro:property name="body_length" value="0.1023" scope="parent"/>
     <xacro:property name="body_color" value="0.25 0.25 0.25 1" scope="parent"/>
-    <xacro:property name="body_collision_radius" value="0.044"/>
+    <xacro:property name="body_collision_size" value="0.1025 0.075 0.115"/>
     <!-- Base Link -->
     <link name="${base_link}"/>
@@ -47,5 +47,5 @@
         <origin xyz="0 0 0" rpy="0 0 0"/>
         <geometry>
-          <cylinder radius="${body_collision_radius}" length="${body_length}"/>
+          <box size="${body_collision_size}"/>
         </geometry>
       </collision>

Commit message: Adjust epick_body box dimensions
Box collision size 0.1025/0.075/0.115 -> 0.07/0.08/0.1 (X/Y/Z).
Visual mesh and body_length kinematic offset still unchanged.

File: epick_description/urdf/epick_body.xacro (robot description, xacro)
@@ -24,5 +24,5 @@
     <xacro:property name="body_length" value="0.1023" scope="parent"/>
     <xacro:property name="body_color" value="0.25 0.25 0.25 1" scope="parent"/>
-    <xacro:property name="body_collision_size" value="0.1025 0.075 0.115"/>
+    <xacro:property name="body_collision_size" value="0.07 0.08 0.1"/>
     <!-- Base Link -->
     <link name="${base_link}"/>
