Commit message: Replace box collision with decimated mesh for epick_body
The 15K-tri visual STL was reduced to 1512 triangles (74 KB) via
the MoveIt Pro `decimate_mesh` script, run twice (maxError 0.5
then 2.0 mm). The collision link now references the decimated
mesh instead of a coarse 0.07x0.08x0.1 m bounding box, giving
FCL contact queries the actual body silhouette while keeping the
tri count two orders of magnitude under the visual.

Co-Authored-By: Claude Opus 4.7 (1M context) <noreply@anthropic.com>

File: epick_description/urdf/epick_body.xacro (robot description, xacro)
@@ -24,5 +24,4 @@
     <xacro:property name="body_length" value="0.1023" scope="parent"/>
     <xacro:property name="body_color" value="0.25 0.25 0.25 1" scope="parent"/>
-    <xacro:property name="body_collision_size" value="0.07 0.08 0.1"/>
     <!-- Base Link -->
     <link name="${base_link}"/>
@@ -45,7 +44,8 @@
       </visual>
       <collision>
-        <origin xyz="0 0 0" rpy="0 0 0"/>
+        <origin xyz="0 0 ${-body_length / 2}" rpy="0 0 0"/>
         <geometry>
-          <box size="${body_collision_size}"/>
+          <mesh filename="package://epick_description/meshes/collision/epick_body.stl"
+            scale="0.001 0.001 0.001"/>
         </geometry>
       </collision>
